File: hardware/prototype.job.brd (EAGLE design)
At the start: 62.2 x 57.2 mm, 32 parts, among them Q3 BS170

Commit message: Smaller PCB, also the placement of the RASPI port has been corrected and the Serial port error
Parts:
- removed 16MHZ: (no value), special:QS
- removed ATMEGA168-20PU: (no value), adafruit:DIL28-3
- removed CANPORT: (no value), con-subd:M09VP
- removed ICSP: AVRISP-6, adafruit:AVRISP
- removed MCP2515-I/P: (no value), MCP2515_MT:DIL18
- removed MCP2551: (no value), micro-philips:DIL08
- removed OSC1: 16MHz, special:QS
- removed RASPI: (no value), con-lstb:MA13-2
- removed RESET: (no value), switch-tact:DTS-6
- removed RXBUF1, RXBUF2: (no value), led:LED5MM
- added IC1: PCA82C251, micro-philips:DIL08
- added IC2: ATMEGA328P-PU, adafruit:DIL28-3
- added ISP1: AVRISP-6, adafruit:AVRISP
- added LED3, LED4: (no value), led:LED5MM
- added Q1, Q2: (no value), special:QS
- added S1: DTS-6, switch-tact:DTS-6
- added SV1: (no value), con-lstb:MA13-2
- added U$1: MCP2515DIL, MCP2515_MT:DIL18
- added X1: (no value), con-subd:M09VP
- moved Q3 23.8 mm to (64.9, 14.9)
- moved R2 23.8 mm to (71.9, 50.9)
- moved R3 23.8 mm to (71.3, 7.57)
- moved R5 23.8 mm to (57.5, 10.9)
- moved C10 23.8 mm to (41.1, 35.9)
- moved C11 23.8 mm to (41.0, 50.6)
- moved C3 23.8 mm to (53.7, 43.3)
- moved C8 23.8 mm to (45.7, 31.4)
- moved C9 23.8 mm to (45.6, 27.9)
- moved C1 23.8 mm to (54.1, 33.9)
- moved C2 23.8 mm to (54.2, 19.0)
- moved C4 23.8 mm to (38.5, 29.8)
- moved C5 23.8 mm to (47.4, 43.2)
- moved C6 23.8 mm to (82.2, 8.22)
- moved D1 23.8 mm to (71.2, 10.4)
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Connections:
- net GND: now also IC1.2, IC2.22, IC2.8, ISP1.6, S1.1, S1.2, SV1.5, U$1.9, X1.3; no longer ATMEGA168-20PU.22, ATMEGA168-20PU.8, CANPORT.3, ICSP.6, MCP2515-I/P.9, MCP2551.2, RASPI.5, RESET.1, RESET.2
- net N$1: now also IC1.1, U$1.1; no longer MCP2515-I/P.1, MCP2551.1
- net N$10: now also IC2.16, U$1.16; no longer ATMEGA168-20PU.16, MCP2515-I/P.16
- net N$11: now also IC2.3; no longer ATMEGA168-20PU.3
- net N$15: now also IC2.19, ISP1.3, U$1.13; no longer ATMEGA168-20PU.19, ICSP.3, MCP2515-I/P.13
- net N$16: now also IC2.9, Q2.2; no longer ATMEGA168-20PU.9, OSC1.2
- net N$17: now also IC2.10, Q2.1; no longer ATMEGA168-20PU.10, OSC1.1
- net N$18: now also IC1.8; no longer MCP2551.8
- net N$19: now also IC2.21; no longer ATMEGA168-20PU.21
- net N$2: now also IC1.4, U$1.2; no longer MCP2515-I/P.2, MCP2551.4
- net N$22: now also SV1.9; no longer RASPI.9
- net N$23: now also IC2.2; no longer ATMEGA168-20PU.2
- net N$24: now also IC2.1, ISP1.5, S1.3, S1.4; no longer ATMEGA168-20PU.1, ICSP.5, RESET.3, RESET.4
- net N$25: now also SV1.2; no longer RASPI.2
- net N$26: now also IC2.18, ISP1.1, U$1.15; no longer ATMEGA168-20PU.18, ICSP.1, MCP2515-I/P.15
- net N$27: now also IC2.17, ISP1.4, U$1.14; no longer ATMEGA168-20PU.17, ICSP.4, MCP2515-I/P.14
- net N$29: now also IC1.6, X1.2; no longer CANPORT.2, MCP2551.6
- net N$3: now also Q1.2, U$1.7; no longer 16MHZ.2, MCP2515-I/P.7
- net N$30: now also IC1.7, X1.7; no longer CANPORT.7, MCP2551.7
- net N$32: now also SV1.7; no longer RASPI.7
- net N$4: now also Q1.1, U$1.8; no longer 16MHZ.1, MCP2515-I/P.8
- net N$5: now also U$1.17; no longer MCP2515-I/P.17
- net N$6: now also LED3.A; no longer RXBUF1.A
- net N$7: now also LED4.A; no longer RXBUF2.A
- net N$8: now also LED4.K, U$1.11; no longer MCP2515-I/P.11, RXBUF2.K
- net N$9: now also LED3.K, U$1.10; no longer MCP2515-I/P.10, RXBUF1.K
- net VCC: now also IC1.3, IC2.20, IC2.7, ISP1.2, SV1.1, U$1.18; no longer ATMEGA168-20PU.20, ATMEGA168-20PU.7, ICSP.2, MCP2515-I/P.18, MCP2551.3, RASPI.1
Routing:
- net N$23: track 50.9 -> 45.0 mm
- net N$25: track 31.6 -> 35.8 mm
- net VCC: track 155.5 -> 152.2 mm
- net GND: track 184.2 -> 180.9 mm
- net N$22: track 31.8 -> 29.3 mm
- net N$24: track 93.4 -> 91.1 mm
- net N$32: track 26.7 -> 24.7 mm
- removed copper zone on layer 1, net N$12
- removed copper zone on layer 16, net N$13
Other:
- outline, holes or cut-outs redrawn
- board text added: "RXBuf0"
- board text added: "RXBuf1"
- board text removed: "By Dimme.net & Leston.me"
